File: pcb/sumoesp.kicad_pcb (KiCad board)
At the start: 2 copper layers, 66 x 66 mm, 29 parts, among them J1 Conn_01x03, J10 Discharge pins, J2 Conn_01x03, J3 USB_B, J4 Charge pins, J5 Photo, J6 Ultrasonic, J7 IR LED, J8 OLED, J9 3.3v step-down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

Commit message: update pcb layout
Parts:
- removed J2: Conn_01x03, Pin_Headers:Pin_Header_Straight_1x03_Pitch2.54mm
- removed R9: 100k, Resistors_THT:R_Axial_DIN0207_L6.3mm_D2.5mm_P7.62mm_Horizontal
- removed the REF** at (173.7, 73.7)
- removed the REF** at (114.3, 133.6)
- removed the REF** at (174.2, 133.6)
- added REF**: MountingHole_3.2mm_M3, Mounting_Holes:MountingHole_3.2mm_M3, F.Cu at (174.0, 73.7)
- added REF**: MountingHole_3.2mm_M3, Mounting_Holes:MountingHole_3.2mm_M3, F.Cu at (174.0, 133.3)
- added REF**: MountingHole_3.2mm_M3, Mounting_Holes:MountingHole_3.2mm_M3, F.Cu at (114.3, 133.3)
- B1: footprint Buttons_Switches_THT:SW_PUSH_6mm -> Buttons_Switches_THT:SW_Tactile_SPST_Angled_PTS645Vx83-2LFS
- J1: value Conn_01x03 -> Servo; footprint Pin_Headers:Pin_Header_Straight_1x03_Pitch2.54mm -> Pin_Headers:Pin_Header_Angled_2x03_Pitch2.54mm
- J10, J9: footprint Socket_Strips:Socket_Strip_Straight_1x03_Pitch2.54mm -> Socket_Strips:Socket_Strip_Angled_1x03_Pitch2.54mm
- J4: footprint Socket_Strips:Socket_Strip_Straight_1x02_Pitch2.54mm -> Socket_Strips:Socket_Strip_Angled_1x02_Pitch2.54mm
- J5, J7: footprint Pin_Headers:Pin_Header_Straight_2x03_Pitch2.54mm -> Pin_Headers:Pin_Header_Angled_2x03_Pitch2.54mm
- J8: moved to F.Cu
- R1, R2: footprint Resistors_THT:R_Axial_DIN0207_L6.3mm_D2.5mm_P7.62mm_Horizontal -> Resistors_THT:R_Axial_DIN0207_L6.3mm_D2.5mm_P10.16mm_Horizontal
- moved B1 15.3 mm to (114.1, 128.3), turned to 90 degrees
- moved J10 12.4 mm to (120.1, 129.0), turned to 180 degrees
- moved J1 11.1 mm to (133.2, 98.3), turned to 0 degrees
- moved R4 11.1 mm to (150.5, 118.1)
- moved R3 11.1 mm to (150.5, 115.6)
- moved R5 10.9 mm to (150.6, 120.7)
- moved J8 10.8 mm to (146.7, 114.3), turned to 180 degrees
- moved Y1 10.8 mm to (127.8, 90.2)
- moved J5 10.7 mm to (164.5, 81.0), turned to 0 degrees
- moved J7 10.6 mm to (161.2, 115.6)
- moved J4 10.3 mm to (120.1, 116.3), turned to 180 degrees
- moved R1 8.70 mm to (124.5, 110.9), turned to 0 degrees
- moved R7 8.03 mm to (162.6, 93.0), turned to 0 degrees
- moved J9 6.66 mm to (145.4, 128.9)
- moved R8 6.66 mm to (162.6, 95.6)
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Connections:
- J1 pad 1: GND -> Net-(J1-Pad1)
- J10 pad 1: GND -> Net-(B1-Pad2)
- J10 pad 3: Net-(B1-Pad2) -> GND
- J4 pad 1: VBUS -> GND
- J4 pad 2: GND -> VBUS
- J5 pad 1: GND -> Net-(J5-Pad1)
- J5 pad 2: Net-(J5-Pad2) -> GND
- J5 pad 3: GND -> Net-(J5-Pad3)
- J5 pad 4: Net-(J5-Pad4) -> GND
- J5 pad 5: GND -> Net-(J5-Pad5)
- J5 pad 6: Net-(J5-Pad6) -> GND
- R1 pad 1: Net-(J1-Pad2) -> Net-(J1-Pad3)
- R2 pad 1: Net-(J2-Pad2) -> Net-(J1-Pad4)
- R6 pad 1: Net-(J5-Pad6) -> Net-(J5-Pad1)
- R7 pad 1: Net-(J5-Pad4) -> Net-(J5-Pad3)
- R8 pad 1: Net-(J5-Pad2) -> Net-(J5-Pad5)
- U1 pad 12: (no net) -> Net-(U1-Pad12)
- U1 pad 13: (no net) -> Net-(U1-Pad13)
- U1 pad 14: (no net) -> Net-(U1-Pad14)
- U1 pad 17: (no net) -> Net-(U1-Pad17)
- U1 pad 18: (no net) -> Net-(U1-Pad18)
- U1 pad 19: (no net) -> Net-(U1-Pad19)
- U1 pad 20: (no net) -> Net-(U1-Pad20)
- U1 pad 21: (no net) -> Net-(U1-Pad21)
- U1 pad 22: (no net) -> Net-(U1-Pad22)
- U1 pad 26: (no net) -> Net-(U1-Pad26)
- U1 pad 27: Net-(J2-Pad3) -> Net-(J1-Pad2)
- U1 pad 28: Net-(J1-Pad3) -> Net-(J1-Pad1)
- U1 pad 29: (no net) -> Net-(U1-Pad29)
- U1 pad 30: (no net) -> Net-(U1-Pad30)
- U1 pad 31: (no net) -> Net-(U1-Pad31)
- U1 pad 32: (no net) -> Net-(U1-Pad32)
- U1 pad 33: (no net) -> Net-(U1-Pad33)
- U1 pad 36: (no net) -> Net-(U1-Pad36)
- U1 pad 37: (no net) -> Net-(U1-Pad37)
- U1 pad 4: Net-(J5-Pad6) -> Net-(J5-Pad1)
- U1 pad 5: Net-(J5-Pad4) -> Net-(J5-Pad3)
- U1 pad 6: Net-(J5-Pad2) -> Net-(J5-Pad5)
- U1 pad 7: (no net) -> Net-(U1-Pad7)
- U1 pad 8: (no net) -> Net-(U1-Pad8)
- U1 pad 9: (no net) -> Net-(U1-Pad9)
- U2 pad 10: (no net) -> Net-(U2-Pad10)
- U2 pad 11: (no net) -> Net-(U2-Pad11)
- U2 pad 12: (no net) -> Net-(U2-Pad12)
- U2 pad 15: (no net) -> Net-(U2-Pad15)
- U2 pad 9: (no net) -> Net-(U2-Pad9)
Routing:
- net Net-(U1-Pad25): track 59.7 -> 79.8 mm
- net Net-(J5-Pad5): track 0.00 -> 20.0 mm
- net Net-(J5-Pad3): track 0.00 -> 17.6 mm
- net Net-(J5-Pad6): track 15.3 -> 0.00 mm
- net +5V: track 64.7 -> 80.0 mm
- net GND: track 15.1 -> 0.00 mm
- net Net-(J5-Pad4): track 14.8 -> 0.00 mm
- net Net-(J5-Pad1): track 0.00 -> 14.3 mm
- net Net-(J5-Pad2): track 14.3 -> 0.00 mm
- net Net-(B1-Pad2): track 17.9 -> 8.19 mm
- net Net-(J1-Pad4): track 0.00 -> 8.35 mm
- net Net-(J1-Pad1): track 0.00 -> 8.26 mm
- net Net-(J8-Pad2): track 10.4 -> 17.8 mm
- net Net-(J2-Pad3): track 7.35 -> 0.00 mm
- net Net-(C1-Pad1): track 18.8 -> 12.9 mm
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Other:
- outline, holes or cut-outs redrawn
- net class Default: clearance 0.2 -> 0.1
- rule trace_clearance: 0.2 -> 0.1
