File: pcb/sumoesp.sch (KiCad schematic (older format))
At the start: 25 parts, among them J1 Conn_01x03, J10 Discharge pins, J2 Conn_01x03, J3 USB_B, J4 Charge pins, J5 Photo, J6 Ultrasonic, J7 IR LED, J8 OLED, J9 3.3v step-down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

Commit message: update pcb layout
Parts:
- removed J1, J2: Conn_01x03, Pin_Headers:Pin_Header_Straight_1x03_Pitch2.54mm, symbol Conn_01x03
- removed R9: 100k, Resistors_THT:R_Axial_DIN0207_L6.3mm_D2.5mm_P7.62mm_Horizontal, symbol R
- added J1: Servo, Pin_Headers:Pin_Header_Angled_2x03_Pitch2.54mm, symbol Conn_02x03_Odd_Even
- B1: footprint Buttons_Switches_THT:SW_PUSH_6mm -> Buttons_Switches_THT:SW_Tactile_SPST_Angled_PTS645Vx83-2LFS
- J10, J9: footprint Socket_Strips:Socket_Strip_Straight_1x03_Pitch2.54mm -> Socket_Strips:Socket_Strip_Angled_1x03_Pitch2.54mm
- J4: footprint Socket_Strips:Socket_Strip_Straight_1x02_Pitch2.54mm -> Socket_Strips:Socket_Strip_Angled_1x02_Pitch2.54mm
- J5, J7: footprint Pin_Headers:Pin_Header_Straight_2x03_Pitch2.54mm -> Pin_Headers:Pin_Header_Angled_2x03_Pitch2.54mm
- R1, R2: footprint Resistors_THT:R_Axial_DIN0207_L6.3mm_D2.5mm_P7.62mm_Horizontal -> Resistors_THT:R_Axial_DIN0207_L6.3mm_D2.5mm_P10.16mm_Horizontal
Other:
- moved on the sheet: R1, R2
